File: VCA/vca.kicad_pcb (KiCad board)
At the start: 2 copper layers, 45.2 x 146.8 mm, 96 parts, among them J1 CVA1, J2 CVA2, J3 OUTA, J4 INA, J5 CV1B, J6 CVB2, J7 OUTB, J8 INB, J9 PWR, Q1 2N3904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

Commit message: Add files via upload
Parts:
- removed G***: LOGO, graphics:errata logo
- removed G***: LOGO, graphics:logo_openhardware
