File: util_LFO/util_LFO.kicad_pcb (KiCad board)
At the start: 2 copper layers, 27.2 x 37.1 mm, 23 parts, among them J1 SQR, J2 TRI, J3 Conn_02x05_Odd_Even, J4 +12, J5 GND, J6 -12, U1 TL072

Commit message: Add files via upload
Parts:
- moved R1 0.05 mm to (102.2, 69.1)
- turned R3 to 180 degrees
Connections:
- RV10 pad : (no net) -> GND
- RV11 pad : (no net) -> GND
- RV11 pad 1: Net-(R3-Pad2) -> Net-(RV10-Pad2)
- RV11 pad 3: Net-(RV10-Pad2) -> Net-(R3-Pad2)
Routing:
- net Net-(RV10-Pad2): track 25.8 -> 10.7 mm
- net Net-(R1-Pad1): track 22.5 -> 18.9 mm
Other:
- board text added: "8K LFO V2.0 Circuit by Tim Parkhurst magsmoke@gmail.com"

Commit message: Add files via upload
Parts:
- moved J6 1.78 mm to (102.1, 59.9)
- moved J4 1.27 mm to (88.9, 59.9)
Routing:
- net -12V: track 53.4 -> 52.7 mm
- net +12v: track 57.5 -> 57.0 mm
Changed lines of the file:
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@@
     (add_net GND)
+  )
+  (module Connector_PinHeader_2.00mm:PinHeader_1x01_P2.00mm_Vertical (layer B.Cu)
+    (at 102.108 59.8805 270)
+    (descr "Through hole straight pin header, 1x01, 2.00mm pitch, single row")
+    (tags "Through hole pin header THT 1x01 2.00mm single row")
+    (fp_text reference J6 (at 0 2.06 270) (layer B.SilkS) hide
+      (effects (font (size 1 1) (thickness 0.15)) (justify mirror))
+    )
+    (fp_text value -12 (at 0 -2.06 270) (layer B.Fab)
+      (effects (font (size 1 1) (thickness 0.15)) (justify mirror))
+    )
+    (fp_line (start -0.5 1) (end 1 1) (layer B.Fab) (width 0.1))
+    (fp_line (start 1 1) (end 1 -1) (layer B.Fab) (width 0.1))
+    (fp_line (start 1 -1) (end -1 -1) (layer B.Fab) (width 0.1))
+    (fp_line (start -1 -1) (end -1 0.5) (layer B.Fab) (width 0.1))
+    (fp_line (start -1 0.5) (end -0.5 1) (layer B.Fab) (width 0.1))
+    (fp_line (start -1.06 -1.06) (end 1.06 -1.06) (layer B.SilkS) (width 0.12))
+    (fp_line (start -1.06 -1) (end -1.06 -1.06) (layer B.SilkS) (width 0.12))
+    (fp_line (start 1.06 -1) (end 1.06 -1.06) (layer B.SilkS) (width 0.12))
+    (fp_line (start -1.06 -1) (end 1.06 -1) (layer B.SilkS) (width 0.12))
+    (fp_line (start -1.06 0) (end -1.06 1.06) (layer B.SilkS) (width 0.12))
+    (fp_line (start -1.06 1.06) (end 0 1.06) (layer B.SilkS) (width 0.12))
+    (fp_line (start -1.5 1.5) (end -1.5 -1.5) (layer B.CrtYd) (width 0.05))
+    (fp_line (start -1.5 -1.5) (end 1.5 -1.5) (layer B.CrtYd) (width 0.05))
+    (fp_line (start 1.5 -1.5) (end 1.5 1.5) (layer B.CrtYd) (width 0.05))
+    (fp_line (start 1.5 1.5) (end -1.5 1.5) (layer B.CrtYd) (width 0.05))
+    (fp_text user %R (at 0 0 180) (layer B.Fab)
+      (effects (font (size 1 1) (thickness 0.15)) (justify mirror))
+    )
+    (pad 1 thru_hole circle (at 0 0 270) (size 1.35 1.35) (drill 0.8) (layers *.Cu *.Mask)
+      (net 5 -12V))
+    (model ${KISYS3DMOD}/Connector_PinHeader_2.00mm.3dshapes/PinHeader_1x01_P2.00mm_Vertical.wrl
+      (at (xyz 0 0 0))
+      (scale (xyz 1 1 1))
+      (rotate (xyz 0 0 0))
+    )
   )
   (module "Custom Parts:Potentiometer_Thonk_Alpha_9mm_Vertical" (layer F.Cu)
@@
   )
   (module Connector_PinHeader_2.00mm:PinHeader_1x01_P2.00mm_Vertical (layer B.Cu)
-    (at 90.17 59.8805 270)
+    (at 88.9 59.8805 270)
     (descr "Through hole straight pin header, 1x01, 2.00mm pitch, single row")
     (tags "Through hole pin header THT 1x01 2.00mm single row")
@@
     (pad 1 thru_hole circle (at 0 0 270) (size 1.35 1.35) (drill 0.8) (layers *.Cu *.Mask)
       (net 3 GND))
-    (model ${KISYS3DMOD}/Connector_PinHeader_2.00mm.3dshapes/PinHeader_1x01_P2.00mm_Vertical.wrl
-      (at (xyz 0 0 0))
-      (scale (xyz 1 1 1))
-      (rotate (xyz 0 0 0))
-    )
-  )
-  (module Connector_PinHeader_2.00mm:PinHeader_1x01_P2.00mm_Vertical (layer B.Cu)
-    (at 100.33 59.8805 270)
-    (descr "Through hole straight pin header, 1x01, 2.00mm pitch, single row")
-    (tags "Through hole pin header THT 1x01 2.00mm single row")
-    (fp_text reference J6 (at 0 2.06 270) (layer B.SilkS) hide
-      (effects (font (size 1 1) (thickness 0.15)) (justify mirror))
-    )
-    (fp_text value -12 (at 0 -2.06 270) (layer B.Fab)
-      (effects (font (size 1 1) (thickness 0.15)) (justify mirror))
-    )
-    (fp_line (start -0.5 1) (end 1 1) (layer B.Fab) (width 0.1))
-    (fp_line (start 1 1) (end 1 -1) (layer B.Fab) (width 0.1))
-    (fp_line (start 1 -1) (end -1 -1) (layer B.Fab) (width 0.1))
-    (fp_line (start -1 -1) (end -1 0.5) (layer B.Fab) (width 0.1))
-    (fp_line (start -1 0.5) (end -0.5 1) (layer B.Fab) (width 0.1))
-    (fp_line (start -1.06 -1.06) (end 1.06 -1.06) (layer B.SilkS) (width 0.12))
-    (fp_line (start -1.06 -1) (end -1.06 -1.06) (layer B.SilkS) (width 0.12))
-    (fp_line (start 1.06 -1) (end 1.06 -1.06) (layer B.SilkS) (width 0.12))
-    (fp_line (start -1.06 -1) (end 1.06 -1) (layer B.SilkS) (width 0.12))
-    (fp_line (start -1.06 0) (end -1.06 1.06) (layer B.SilkS) (width 0.12))
-    (fp_line (start -1.06 1.06) (end 0 1.06) (layer B.SilkS) (width 0.12))
-    (fp_line (start -1.5 1.5) (end -1.5 -1.5) (layer B.CrtYd) (width 0.05))
-    (fp_line (start -1.5 -1.5) (end 1.5 -1.5) (layer B.CrtYd) (width 0.05))
-    (fp_line (start 1.5 -1.5) (end 1.5 1.5) (layer B.CrtYd) (width 0.05))
-    (fp_line (start 1.5 1.5) (end -1.5 1.5) (layer B.CrtYd) (width 0.05))
-    (fp_text user %R (at 0 0 180) (layer B.Fab)
-      (effects (font (size 1 1) (thickness 0.15)) (justify mirror))
-    )
-    (pad 1 thru_hole circle (at 0 0 270) (size 1.35 1.35) (drill 0.8) (layers *.Cu *.Mask)
-      (net 5 -12V))
     (model ${KISYS3DMOD}/Connector_PinHeader_2.00mm.3dshapes/PinHeader_1x01_P2.00mm_Vertical.wrl
       (at (xyz 0 0 0))
@@
   (segment (start 88.878 93.24) (end 89.916 92.202) (width 0.45) (layer F.Cu) (net 4))
   (segment (start 85.852 93.24) (end 88.878 93.24) (width 0.45) (layer F.Cu) (net 4))
-  (segment (start 85.064999 64.985501) (end 90.17 59.8805) (width 0.45) (layer F.Cu) (net 4))
+  (segment (start 85.064999 63.715501) (end 88.9 59.8805) (width 0.45) (layer F.Cu) (net 4))
   (segment (start 89.916 89.662) (end 85.064999 84.810999) (width 0.45) (layer F.Cu) (net 4))
-  (segment (start 85.064999 84.810999) (end 85.064999 64.985501) (width 0.45) (layer F.Cu) (net 4))
+  (segment (start 85.064999 84.810999) (end 85.064999 63.715501) (width 0.45) (layer F.Cu) (net 4))
   (segment (start 100.1665 83.439) (end 100.584 83.0215) (width 0.45) (layer B.Cu) (net 5))
   (segment (start 98.204 84.6395) (end 96.9915 85.852) (width 0.45) (layer B.Cu) (net 5))
@@
   (segment (start 101.144913 88.798401) (end 100.939599 88.798401) (width 0.45) (layer F.Cu) (net 5))
   (segment (start 106.023001 83.920313) (end 101.144913 88.798401) (width 0.45) (layer F.Cu) (net 5))
-  (segment (start 106.023001 66.528095) (end 106.023001 83.920313) (width 0.45) (layer F.Cu) (net 5))
-  (segment (start 100.33 60.835094) (end 106.023001 66.528095) (width 0.45) (layer F.Cu) (net 5))
-  (segment (start 100.33 59.8805) (end 100.33 60.835094) (width 0.45) (layer F.Cu) (net 5))
+  (segment (start 106.023001 64.750095) (end 106.023001 83.920313) (width 0.45) (layer F.Cu) (net 5))
+  (segment (start 102.108 60.835094) (end 106.023001 64.750095) (width 0.45) (layer F.Cu) (net 5))
+  (segment (start 102.108 59.8805) (end 102.108 60.835094) (width 0.45) (layer F.Cu) (net 5))
   (segment (start 101.6 84.5455) (end 101.6 86.076) (width 0.3) (layer B.Cu) (net 7))
   (segment (start 103.124 83.0215) (end 101.6 84.5455) (width 0.3) (layer B.Cu) (net 7))
